File: untitled2.kicad_sch (KiCad schematic)
At the start: 0 parts

Commit message: additional chamges
Other:
- company: (none) -> Andy McCann KA3KAF and Doug McCann KA3KAG
Changed lines of the file:
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@@
 (kicad_sch (version 20211123) (generator eeschema)
-  (paper "A")
+  (paper "USLegal")
+  (title_block
+    (company "Andy McCann KA3KAF and Doug McCann KA3KAG")
+    (comment 1 "Terry White K7TAU")
+    (comment 2 "Wes Hayward W7ZOI")
+    (comment 3 "Original Design By:")
+  )
 )
