File: W7ZOI Spectrum Analyzer.kicad_sch (KiCad schematic)
At the start: 0 parts

Commit message: additional chamges
Other:
- sheet Not yet used renamed IF and Log Amplifier
- sheet TImeBase renamed TimeBase
- sheet IF and Log Amplifier: file untitled.kicad_sch -> if_log_amplifier.kicad_sch
- title: TimeBase -> Spectrum Analyzer

Commit message: test deletion
Other:
- sheet Unused renamed Resolution Filters
- sheet Resolution Filters: file untitled2.kicad_sch -> Resolution Filters.kicad_sch
Changed lines of the file:
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@@
   (title_block
     (title "Spectrum Analyzer")
-    (date "2022-05-28")
-    (rev "0.2")
+    (date "2022-05-30")
+    (rev "0.3")
     (company "Andy McCann KA3KAF and Doug McCann KA3KAG")
-    (comment 1 "Terry White K7TAU")
-    (comment 2 "Wes Hayward W7ZOI")
-    (comment 3 "Original Design By:")
+    (comment 2 "Terry White K7TAU")
+    (comment 3 "Wes Hayward W7ZOI")
+    (comment 4 "Original Design By:")
   )
-  (image (at 181.61 55.88) (scale 0.829898)
+  (image (at 154.94 54.61) (scale 0.801488)
     (data
       iVBORw0KGgoAAAANSUhEUgAAB8AAAASGCAIAAADZyyOxAAAAA3NCSVQICAjb4U/gAAAACXBIWXMA
@@
     )
   )
-  (sheet (at 22.86 72.39) (size 33.02 39.37) (fields_autoplaced)
-    (stroke (width 0.1524) (type solid) (color 0 0 0 0))
-    (fill (color 0 0 0 0.0000))
-    (property "Sheet name" "Unused" (id 0) (at 22.86 71.6784 0)
-      (effects (font (size 1.27 1.27)) (justify left bottom))
+  (sheet (at 166.37 120.65) (size 33.02 39.37) (fields_autoplaced)
+    (stroke (width 0.254) (type solid) (color 255 0 255 1))
+    (fill (color 132 132 0 1.0000))
+    (property "Sheet name" "Resolution Filters" (id 0) (at 166.37 119.9384 0)
+      (effects (font (size 2.54 2.54)) (justify left bottom))
     )
-    (property "Sheet file" "untitled2.kicad_sch" (id 1) (at 22.86 112.3446 0)
-      (effects (font (size 1.27 1.27)) (justify left top))
+    (property "Sheet file" "Resolution Filters.kicad_sch" (id 1) (at 166.37 160.6046 0)
+      (effects (font (size 1.905 1.905)) (justify left top))
     )
   )
-  (sheet (at 220.98 115.57) (size 33.02 39.37)
+  (sheet (at 240.03 120.65) (size 33.02 39.37)
     (stroke (width 0.254) (type solid) (color 255 0 255 1))
     (fill (color 132 132 0 1.0000))
-    (property "Sheet name" "IF and Log Amplifier" (id 0) (at 218.44 113.03 0)
+    (property "Sheet name" "IF and Log Amplifier" (id 0) (at 237.49 118.11 0)
       (effects (font (size 2.54 2.54)) (justify left bottom))
     )
-    (property "Sheet file" "if_log_amplifier.kicad_sch" (id 1) (at 215.9 157.48 0)
+    (property "Sheet file" "if_log_amplifier.kicad_sch" (id 1) (at 234.95 162.56 0)
       (effects (font (size 1.905 1.905)) (justify left top))
     )
@@
       (reference "C406") (unit 1) (value "100u") (footprint "Capacitor_THT:CP_Axial_L11.0mm_D6.0mm_P18.00mm_Horizontal")
     )
+    (path "/1213119d-b3ea-47c8-aaf6-ecc398bfbb00/102a6993-b6e6-44ab-89e4-1c06022fe226"
+      (reference "C?") (unit 1) (value "C_Small") (footprint "")
+    )
+    (path "/1213119d-b3ea-47c8-aaf6-ecc398bfbb00/135f8e46-3647-446e-983d-ca74361cba41"
+      (reference "C?") (unit 1) (value "C_Small") (footprint "")
+    )
+    (path "/1213119d-b3ea-47c8-aaf6-ecc398bfbb00/20b5bf70-e4f8-4af3-a29d-328d67b94ee4"
+      (reference "C?") (unit 1) (value "C_Small") (footprint "")
+    )
+    (path "/1213119d-b3ea-47c8-aaf6-ecc398bfbb00/25d340ff-64e6-4e47-8537-6ea572896d15"
+      (reference "C?") (unit 1) (value "C_Small") (footprint "")
+    )
+    (path "/1213119d-b3ea-47c8-aaf6-ecc398bfbb00/3984c9a0-ac94-4cfc-aa87-2b9b9a5716fe"
+      (reference "C?") (unit 1) (value "C_Small") (footprint "")
+    )
+    (path "/1213119d-b3ea-47c8-aaf6-ecc398bfbb00/3ab4a587-3f66-48c4-ae40-b64ac0b69dcb"
+      (reference "C?") (unit 1) (value "C_Small") (footprint "")
+    )
+    (path "/1213119d-b3ea-47c8-aaf6-ecc398bfbb00/3bee70c9-2f50-4eb6-9a8f-df584e12a895"
+      (reference "C?") (unit 1) (value "C_Small") (footprint "")
+    )
+    (path "/1213119d-b3ea-47c8-aaf6-ecc398bfbb00/40c8ffaf-cce9-4a86-882b-7e5b7d105be4"
+      (reference "C?") (unit 1) (value "C_Small") (footprint "")
+    )
+    (path "/1213119d-b3ea-47c8-aaf6-ecc398bfbb00/6c05f317-9b48-44ed-b337-51f5d38b951b"
+      (reference "C?") (unit 1) (value "C_Small") (footprint "")
+    )
+    (path "/1213119d-b3ea-47c8-aaf6-ecc398bfbb00/98baa52c-33e4-472b-9cde-bef009b48d60"
+      (reference "C?") (unit 1) (value "C_Small") (footprint "")
+    )
+    (path "/1213119d-b3ea-47c8-aaf6-ecc398bfbb00/9d053ddf-727f-4ac3-99a4-04f1659f5de2"
+      (reference "C?") (unit 1) (value "C_Small") (footprint "")
+    )
+    (path "/1213119d-b3ea-47c8-aaf6-ecc398bfbb00/ab7e4f62-073d-4dfd-8975-5f0733fb7ad5"
+      (reference "C?") (unit 1) (value "C_Small") (footprint "")
+    )
+    (path "/1213119d-b3ea-47c8-aaf6-ecc398bfbb00/cf0bef72-ca14-4e69-be35-1f112576b0ca"
+      (reference "C?") (unit 1) (value "C_Small") (footprint "")
+    )
+    (path "/1213119d-b3ea-47c8-aaf6-ecc398bfbb00/d6db0d3a-db08-4423-a8b8-b50569d21b1c"
+      (reference "C?") (unit 1) (value "C_Small") (footprint "")
+    )
+    (path "/1213119d-b3ea-47c8-aaf6-ecc398bfbb00/dec87add-cf42-4a5e-81a0-0ad45593dd87"
+      (reference "C?") (unit 1) (value "C_Small") (footprint "")
+    )
+    (path "/1213119d-b3ea-47c8-aaf6-ecc398bfbb00/ef81a283-08ef-4b13-b7da-40db626e5a5b"
+      (reference "C?") (unit 1) (value "C_Small") (footprint "")
+    )
     (path "/91afdbb9-c6d6-4a76-a186-be607f7c2a6b/f72c35a8-841a-4e17-9a61-84fe02cc96f1"
       (reference "D301") (unit 1) (value "1N4152") (footprint "Diode_THT:D_DO-35_SOD27_P7.62mm_Horizontal")
@@
       (reference "J404") (unit 1) (value "Jack-DC") (footprint "SnapEDA Library:CUI_PJ-007")
     )
+    (path "/1213119d-b3ea-47c8-aaf6-ecc398bfbb00/5c2fd91a-2547-4d62-bb9f-a69cddcb397b"
+      (reference "J?") (unit 1) (value "Conn_Coaxial") (footprint "")
+    )
+    (path "/1213119d-b3ea-47c8-aaf6-ecc398bfbb00/61ea7daf-b2f9-4c78-976f-bdf878ac8cb7"
+      (reference "J?") (unit 1) (value "Conn_Coaxial") (footprint "")
+    )
     (path "/91afdbb9-c6d6-4a76-a186-be607f7c2a6b/18811d97-2857-4d12-8c0c-c5980a41d13f"
       (reference "L301") (unit 1) (value "1.05u") (footprint "")
     )
+    (path "/1213119d-b3ea-47c8-aaf6-ecc398bfbb00/1a36491f-08e2-47d5-b521-bf448d8049f6"
+      (reference "L?") (unit 1) (value "L") (footprint "")
+    )
+    (path "/1213119d-b3ea-47c8-aaf6-ecc398bfbb00/8cc51c4c-4a41-4ae7-8b11-5c3ed2de1af6"
+      (reference "L?") (unit 1) (value "L") (footprint "")
+    )
+    (path "/1213119d-b3ea-47c8-aaf6-ecc398bfbb00/a6b36c9f-b964-489e-a093-3510930923cc"
+      (reference "L?") (unit 1) (value "L") (footprint "")
+    )
+    (path "/1213119d-b3ea-47c8-aaf6-ecc398bfbb00/d4ef91f2-131b-412b-8ac0-c9fd0109137b"
+      (reference "L?") (unit 1) (value "L") (footprint "")
+    )
     (path "/91afdbb9-c6d6-4a76-a186-be607f7c2a6b/efa65d84-4d33-4d24-8ecd-912f1b43323c"
       (reference "R2") (unit 1) (value "10k") (footprint "")
@@
       (reference "R429") (unit 1) (value "470") (footprint "Resistor_THT:R_Axial_DIN0207_L6.3mm_D2.5mm_P7.62mm_Horizontal")
     )
+    (path "/1213119d-b3ea-47c8-aaf6-ecc398bfbb00/008b2ae2-156b-4406-90d0-c10b5844ed31"
+      (reference "R?") (unit 1) (value "R_Small_US") (footprint "")
+    )
+    (path "/1213119d-b3ea-47c8-aaf6-ecc398bfbb00/2f602ec4-7a44-40e6-a667-94f41bbf5036"
+      (reference "R?") (unit 1) (value "R_Small_US") (footprint "")
+    )
+    (path "/1213119d-b3ea-47c8-aaf6-ecc398bfbb00/d4c14093-5e8f-4860-837b-b9fff0fa8797"
+      (reference "R?") (unit 1) (value "R_Small_US") (footprint "")
+    )
     (path "/91afdbb9-c6d6-4a76-a186-be607f7c2a6b/cb3863cc-5c2c-43a7-916e-57f00a70081c"
