File: Timebase.kicad_sch (KiCad schematic)
At the start: 57 parts

Commit message: additional chamges
Parts:
- added H1, H2, H3, H4: MountingHole_Pad, MountingHole:MountingHole_2.7mm_M2.5_DIN965_Pad_TopOnly, symbol Mechanical:MountingHole_Pad
- added J402, J404: Jack-DC, SnapEDA Library:CUI_PJ-007, symbol Connector:Jack-DC
- added J8, J9: Conn_Coaxial, SnapEDA Library:TE_5-1634503-1, symbol Connector:Conn_Coaxial
- C401: renamed from C?; footprint (none) -> Capacitor_THT:C_Radial_D4.0mm_H5.0mm_P1.50mm
- C402, C403, C404, C405, C406: renamed from C?; footprint (none) -> Capacitor_THT:CP_Axial_L11.0mm_D6.0mm_P18.00mm_Horizontal
- D403, D406: renamed from D?; footprint (none) -> Diode_THT:D_DO-35_SOD27_P7.62mm_Horizontal
- R3, R4, R5, R6: renamed from R?; footprint (none) -> Connector_Wire:SolderWire-0.127sqmm_1x03_P3.7mm_D0.48mm_OD1mm
- R401, R402, R403, R404, R405, R406, R407, R408, R409, R410, R411, R412, R413, R414, R415, R416, R417, R418, R419, R421, R422, R423, R425, R426, R427, R428, R429: renamed from R?; footprint (none) -> Resistor_THT:R_Axial_DIN0207_L6.3mm_D2.5mm_P7.62mm_Horizontal
- R420: renamed from R?; footprint (none) -> Potentiometer_THT:Potentiometer_Bourns_3296W_Vertical; Spice_Lib_File Pot5.lib -> Pot6.lib; Spice_Model pot_lin5 -> pot_lin6
- R424: renamed from R?; footprint (none) -> Potentiometer_THT:Potentiometer_Bourns_3296W_Vertical; Spice_Lib_File Pot6.lib -> Pot5.lib; Spice_Model pot_lin6 -> pot_lin5
- U401, U402, U403: renamed from U?; value TL072 -> LM358; footprint (none) -> SnapEDA Library:DIP794W45P254L959H508Q8; symbol Amplifier_Operational:TL072 -> Amplifier_Operational:LM358
- V401, V402: renamed from V?; footprint (none) -> SnapEDA Library:CUI_PJ-009A
- gave numbers to parts that had none: 5
Connections:
- net GND: now also H1.1, H2.1, H3.1, H4.1, J402.2, J404.2, J8.2 (Ext), J9.2 (Ext)
- net Out: now also J9.1 (In)
- net V+15: now also J402.1
- net VCO_Out: now also J8.1 (In)
- net R6Pin1 renamed V-15
- net V-15: now also J404.1
Other:
- note added: ".param Rt=10k set=0.9 .param Rt2=10k set2=0.5 .param Rt3=5k set3=0.5 .param Rt4=10k set4=0.9 .param Rt5=5k set5=0.9 .param Rt6=5k set6=0.5"
- note added: "Mechanicals"
- note removed: ".param Rt=10k set=0.5 .param Rt2=10k set2=0.5 .param Rt3=5k set3=0.5 .param Rt4=10k set4=0.5 .param Rt5=5k set5=0.5 .param Rt6=5k set6=0.5"
- company: (none) -> Andy McCann KA3KAF and Doug McCann KA3KAG
- title: (none) -> Spectrum Analyzer
- moved on the sheet: C401, C402, C403, C404, C405, C406, D401, D402, D403, D404, D405, D406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
