File: 15v-power-supply.kicad_sch (KiCad schematic)
At the start: 23 parts, among them J801 Screw_Terminal_01x03, P801 120VAC, T801 XFORMER, U801 LM7815, U802 LM7915

Commit message: if and log amp routing and 3d model
Parts:
- removed C801: 0.22u, Capacitor_THT:C_Axial_L5.1mm_D3.1mm_P7.50mm_Horizontal, symbol Device:C_Small
- removed C802, C803, C810, C811: 6800u, symbol Device:C_Polarized_Small_US
- removed C804, C805: 6.8u, symbol Device:C_Small
- removed C806, C807, C808, C809: 0.01u, symbol Device:C_Small
- removed D801, D802, D803, D804: 1n5060, DO15-12, symbol 1N5060GP:1N5060GP
- removed F801: 0.5A, symbol Device:Fuse
- removed J801: Screw_Terminal_01x03, TerminalBlock_4Ucon:TerminalBlock_4Ucon_1x03_P3.50mm_Horizontal, symbol Connector:Screw_Terminal_01x03
- removed P801: 120VAC, symbol Connector:Conn_WallPlug_Earth
- removed R801, R802: 2.2k, symbol Device:R_Small_US
- removed T801: XFORMER, symbol Device:Transformer_1P_2S
- removed U801: LM7815, symbol Regulator_Linear:L7815
- removed U802: LM7915, symbol Regulator_Linear:L7915
- added C901: 0.22u, Capacitor_THT:C_Rect_L4.6mm_W5.5mm_P2.50mm_MKS02_FKP02, symbol Device:C_Small
- added C902, C903, C910, C911: 6800u, 15v-supply:6800u-UVR1H682MRD6, symbol Device:C_Polarized_Small_US
- added C904, C905: 6.8u, Capacitor_THT:CP_Radial_D5.0mm_P2.50mm, symbol Device:C_Small
- added C906, C907, C908, C909: 0.01u, 15v-supply:C_Rect_L6.0mm_W3.5mm_P3.5mm_QYX1H103JTP3TA, symbol Device:C_Small
- added D901, D902, D903, D904: (no value), symbol 1N5060GP:1N5060GP
- added F901: (no value), symbol Device:Fuse
- added H901, H902, H903, H904: MountingHole, MountingHole:MountingHole_3.2mm_M3, symbol Mechanical:MountingHole
- added J901: (no value), symbol terminal-block:691103110003
- added J902: Terminal Block, 15v-supply:terminal-block-691103110003, symbol terminal-block:691103110003
- added P901: 120VAC, symbol Connector:Conn_WallPlug_Earth
- added R901, R902: 2.2k, Resistor_THT:R_Axial_DIN0309_L9.0mm_D3.2mm_P12.70mm_Horizontal, symbol Device:R_Small_US
- added SW901: (no value), symbol Switch:SW_SPST
- added T901: (no value), symbol Device:Transformer_1P_2S
- added U901: (no value), symbol Regulator_Linear:L7815
- added U902: (no value), symbol Regulator_Linear:L7915
Connections:
- net 7815 IN: now also C906.1, C908.1, C910.1, D901.2 (Anode), D903.2 (Anode), U901.1 (IN)
- net 7915 IN: now also C907.2, C909.2, C911.2, D902.1 (Cathode), D904.1 (Cathode), U902.2 (VI)
- net GND: now also C902.2, C903.1, C904.2, C905.1, C910.2, C911.1, J901.2, J902.2, P901.3 (EARTH), R901.2, R902.1, T901.4 (SB), T901.5 (SC), U901.2 (GND), U902.1 (GND)
- net TRAN OUT1: now also C906.2, C907.1, D901.1 (Cathode), D902.2 (Anode), J901.1, T901.3 (SA)
- net TRAN OUT2: now also C908.2, C909.1, D903.1 (Cathode), D904.2 (Anode), J901.3, T901.6 (SD)
- net VCC: now also P901.1 (AC_P), SW901.1 (A)
- new net: C901.1, F901.2, T901.1 (AA)
- new net: C901.2, P901.2 (AC_N), T901.2 (AB)
- new net: F901.1, SW901.2 (B)
- new net +15 REGULATED: C902.1, C904.1, J902.1, R901.1, U901.3 (OUT)
- new net -15 REGULATED: C903.2, C905.2, J902.3, R902.2, U902.3 (VO)
Other:
- note added: "Earth Ground"
- note added: "Spice Simulation Command"
- note removed: "+15 REGULATED"
- note removed: "-15 REGULATED"
