File: resolution-filters/resolution-filters/resolution-filters.kicad_pcb (KiCad board)
At the start: 2 copper layers, 91.7 x 48.8 mm, 61 parts, among them J501 Conn_Coaxial, J502 691137710002, J503 Conn_Coaxial, K501 G5V-1, K502 G5V-1, T501 Transformer_1P_1S, T502 Transformer_1P_1S, Y501 10.7MHz, Y502 10.7MHz, Y503 10.7MHz, Y504 10.7MHz

Commit message: resolution-filters.kicad_pcb updated
Parts:
- removed the TP505 at (146.1, 94.5)
- added TP506: TestPoint, TestPoint:TestPoint_Pad_D2.0mm, F.Cu at (146.2, 94.6)
- C504: renamed from C507; value 120p -> 100p
- C507: renamed from C512; value 180p -> 150p
- C510: renamed from C517; value 180p -> 150p
- C513: renamed from C522; value 120p -> 100p
- renumbered C504 to C503, C509 to C505, C510 to C506, C514 to C508, C515 to C509, C519 to C511, C520 to C512, C523 to C514, C524 to C515, C506 to C516, C521 to C517, C505 to C518, C508 to C519, C511 to C520, C513 to C521, C516 to C522, C518 to C523, J503 to J502, J502 to J503, R502 to R501, R501 to R502, R508 to R505, R509 to R506, R510 to R507, R511 to R508, R505 to R509, R506 to R510, R507 to R511, TP502 to TP501, TP503 to TP502, TP504 to TP503, TP506 to TP504, TP501 to TP505
Connections:
- C501 pad 1: Net-(C501-Pad1) -> /300kHz In
- C502 pad 1: Net-(C501-Pad2) -> /300kHz In
- C503 pad 1: Net-(C501-Pad1) -> Net-(C501-Pad2)
- C504 pad 1: Net-(C501-Pad1) -> Net-(C501-Pad2)
- C505 pad 1: Net-(C501-Pad1) -> Net-(C501-Pad2)
- C514 pad 2: Net-(C523-Pad2) -> Net-(C514-Pad2)
- C515 pad 1: Net-(C523-Pad2) -> Net-(C514-Pad2)
- C518 pad 1: Net-(C505-Pad1) -> Net-(C518-Pad1)
- C519 pad 1: Net-(C508-Pad1) -> Net-(C519-Pad1)
- C521 pad 1: Net-(C513-Pad1) -> Net-(C521-Pad1)
- C522 pad 1: Net-(C516-Pad1) -> Net-(C522-Pad1)
- K501 pad 1: Net-(C501-Pad2) -> /300kHz In
- K501 pad 10: Net-(K501-Pad10) -> /30kHz In
- K502 pad 1: Net-(K502-Pad1) -> /300kHz Out
- K502 pad 10: Net-(K502-Pad10) -> /30Khz Out
- L501 pad 1: Net-(C501-Pad1) -> Net-(C501-Pad2)
- R506 pad 1: Net-(K502-Pad1) -> Net-(C514-Pad2)
- R507 pad 1: Net-(K502-Pad1) -> Net-(C514-Pad2)
- R507 pad 2: Net-(C523-Pad2) -> /300kHz Out
- R508 pad 1: Net-(C523-Pad2) -> /300kHz Out
- R510 pad 2: Net-(C513-Pad1) -> Net-(C521-Pad1)
- R511 pad 1: Net-(C513-Pad1) -> Net-(C521-Pad1)
- T501 pad 1: Net-(K501-Pad10) -> GND
- T501 pad 2: GND -> /30kHz In
- T501 pad 4: Net-(C505-Pad1) -> Net-(C518-Pad1)
- T502 pad 1: Net-(K502-Pad10) -> GND
- T502 pad 2: GND -> /30Khz Out
- TP501 pad 1: Net-(K501-Pad10) -> /30kHz In
- TP504 pad 1: Net-(C523-Pad2) -> /30Khz Out
- TP505 pad 1: Net-(C501-Pad2) -> /300kHz In
- Y501 pad 1: Net-(C505-Pad1) -> Net-(C519-Pad1)
- Y501 pad 3: Net-(C508-Pad1) -> Net-(C518-Pad1)
- Y502 pad 1: Net-(C508-Pad1) -> Net-(C519-Pad1)
- Y503 pad 1: Net-(C513-Pad1) -> Net-(C522-Pad1)
- Y503 pad 3: Net-(C516-Pad1) -> Net-(C521-Pad1)
- Y504 pad 1: Net-(C516-Pad1) -> Net-(C522-Pad1)
Routing:
- net Net-(C523-Pad2): track 61.9 -> 0.00 mm
- net Net-(K502-Pad10): track 46.6 -> 0.00 mm
- net /30Khz Out: track 0.00 -> 46.4 mm
- net /300kHz Out: track 0.00 -> 44.0 mm
- net Net-(C516-Pad1): track 32.8 -> 0.00 mm
- net Net-(C513-Pad1): track 30.1 -> 0.00 mm
- net Net-(C522-Pad1): track 0.00 -> 30.0 mm
- net Net-(C505-Pad1): track 29.9 -> 0.00 mm
- net Net-(C518-Pad1): track 0.00 -> 29.4 mm
- net Net-(C501-Pad1): track 28.9 -> 0.00 mm
- net Net-(C519-Pad1): track 0.00 -> 27.6 mm
- net /300kHz In: track 0.00 -> 26.3 mm
- net Net-(C521-Pad1): track 0.00 -> 26.2 mm
- net Net-(C514-Pad2): track 0.00 -> 24.2 mm
- net Net-(C508-Pad1): track 24.1 -> 0.00 mm
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