File: resolution-filters/resolution-filters/resolution-filters.kicad_pcb (KiCad board)
At the start: 2 copper layers, 91.7 x 48.8 mm, 61 parts, among them J501 Conn_Coaxial, J502 Conn_Coaxial, J503 691137710002, K501 G5V-1, K502 G5V-1, T501 Transformer_1P_1S, T502 Transformer_1P_1S, Y501 10.7MHz, Y502 10.7MHz, Y503 10.7MHz, Y504 10.7MHz

Commit message: resolution filter minor changes
Parts:
- J503: value 691137710002 -> Terminal Block
