File: hierarchical-schematic/15v-power-supply.kicad_sch (KiCad schematic)
At the start: 25 parts, among them J1101 Terminal Block, J1102 Terminal Block, P1101 120VAC, SW1101 SW_SPST, T1101 XFORMER, U1101 LM7815, U1102 LM7915

Commit message: hierarchical schematic updated to pass erc
Parts:
- D1101, D1102, D1103, D1104: footprint Diode_THT:D_DO-41_SOD81_P7.62mm_Horizontal -> DO15-12; symbol 1N5060GP:1N5060GP -> spectrum analyzer:1N5060GP
- J1101, J1102: footprint 15v-supply:terminal-block-691103110003 -> 691103110003; symbol terminal-block:691103110003 -> spectrum analyzer:691103110003
Other:
- note added: "Common"
Changed lines of the file:
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@@
   (junction (at 180.34 45.72) (diameter 0) (color 0 0 0 0)
   )
-  (junction (at 144.78 50.8) (diameter 0) (color 0 0 0 0)
-  )
   (junction (at 186.69 157.48) (diameter 0) (color 0 0 0 0)
   )
@@
     (stroke (width 0) (type default) (color 0 0 0 0))
   )
+  (wire (pts (xy 186.69 130.81) (xy 245.11 130.81))
+    (stroke (width 0) (type default) (color 0 0 0 0))
+  )
   (wire (pts (xy 107.95 157.48) (xy 77.47 157.48))
     (stroke (width 0) (type default) (color 0 0 0 0))
@@
     (stroke (width 0) (type default) (color 0 0 0 0))
   )
-  (wire (pts (xy 144.78 50.8) (xy 156.21 50.8))
+  (wire (pts (xy 137.16 50.8) (xy 156.21 50.8))
     (stroke (width 0) (type default) (color 0 0 0 0))
   )
@@
     (stroke (width 0) (type default) (color 0 0 0 0))
   )
-  (wire (pts (xy 186.69 130.81) (xy 245.11 130.81))
-    (stroke (width 0) (type default) (color 0 0 0 0))
-  )
   (wire (pts (xy 116.84 45.72) (xy 113.03 45.72))
     (stroke (width 0) (type default) (color 0 0 0 0))
@@
     (stroke (width 0) (type default) (color 0 0 0 0))
   )
-  (wire (pts (xy 137.16 50.8) (xy 144.78 50.8))
-    (stroke (width 0) (type default) (color 0 0 0 0))
-  )
   (wire (pts (xy 245.11 128.27) (xy 238.76 128.27))
     (stroke (width 0) (type default) (color 0 0 0 0))
   )
-  (wire (pts (xy 144.78 39.37) (xy 144.78 50.8))
-    (stroke (width 0) (type default) (color 0 0 0 0))
-  )
   (wire (pts (xy 180.34 45.72) (xy 154.94 45.72))
     (stroke (width 0) (type default) (color 0 0 0 0))
@@
     (effects (font (size 1.27 1.27)) (justify left bottom))
   )
+  (text "Common" (at 224.79 129.54 0)
+    (effects (font (size 1.27 1.27)) (justify left bottom))
+  )
   (text "50V" (at 201.295 74.93 0)
     (effects (font (size 1.27 1.27)) (justify left bottom))
@@
   )
   (label "7915 IN" (at 93.98 157.48 0)
-    (effects (font (size 1.27 1.27)) (justify left bottom))
-  )
-  (label "Common" (at 232.41 130.81 90)
     (effects (font (size 1.27 1.27)) (justify left bottom))
   )
@@
     (pin "1")
     (pin "2")
-  )
-  (symbol (lib_id "power:PWR_FLAG") (at 144.78 39.37 0) (unit 1)
-    (in_bom yes) (on_board yes) (fields_autoplaced)
-    (property "Reference" "#FLG01102" (id 0) (at 144.78 37.465 0)
-      (effects (font (size 1.27 1.27)) hide)
-    )
-    (property "Value" "PWR_FLAG" (id 1) (at 144.78 34.29 0))
-    (property "Footprint" "" (id 2) (at 144.78 39.37 0)
-      (effects (font (size 1.27 1.27)) hide)
-    )
-    (property "Datasheet" "~" (id 3) (at 144.78 39.37 0)
-      (effects (font (size 1.27 1.27)) hide)
-    )
-    (pin "1")
   )
   (symbol (lib_id "power:GND") (at 76.2 59.69 0) (unit 1)
@@
     (pin "2")
   )
-  (symbol (lib_id "1N5060GP:1N5060GP") (at 217.17 71.12 90) (unit 1)
+  (symbol (lib_id "spectrum analyzer:1N5060GP") (at 217.17 71.12 90) (unit 1)
     (in_bom yes) (on_board yes) (fields_autoplaced)
     (property "Reference" "D1104" (id 0) (at 220.98 69.8499 90)
@@
       (effects (font (size 1.27 1.27)) (justify right))
     )
-    (property "Footprint" "Diode_THT:D_DO-41_SOD81_P7.62mm_Horizontal" (id 2) (at 217.17 71.12 0)
+    (property "Footprint" "DO15-12" (id 2) (at 219.71 78.74 0)
       (effects (font (size 1.27 1.27)) (justify left bottom) hide)
     )
@@
     (pin "2")
   )
-  (symbol (lib_name "1N5060GP_3") (lib_id "1N5060GP:1N5060GP") (at 180.34 71.12 90) (unit 1)
+  (symbol (lib_name "1N5060GP_3") (lib_id "spectrum analyzer:1N5060GP") (at 180.34 71.12 90) (unit 1)
     (in_bom yes) (on_board yes) (fields_autoplaced)
     (property "Reference" "D1102" (id 0) (at 184.15 69.8499 90)
@@
       (effects (font (size 1.27 1.27)) (justify right))
     )
-    (property "Footprint" "Diode_THT:D_DO-41_SOD81_P7.62mm_Horizontal" (id 2) (at 180.34 71.12 0)
+    (property "Footprint" "DO15-12" (id 2) (at 182.88 78.74 0)
       (effects (font (size 1.27 1.27)) (justify left bottom) hide)
     )
@@
     (pin "2")
   )
-  (symbol (lib_id "terminal-block:691103110003") (at 161.29 50.8 270) (unit 1)
+  (symbol (lib_id "spectrum analyzer:691103110003") (at 161.29 50.8 270) (unit 1)
     (in_bom yes) (on_board yes) (fields_autoplaced)
     (property "Reference" "J1101" (id 0) (at 162.56 49.5299 90)
@@
       (effects (font (size 1.27 1.27)) (justify left))
     )
-    (property "Footprint" "15v-supply:terminal-block-691103110003" (id 2) (at 161.29 50.8 0)
+    (property "Footprint" "691103110003" (id 2) (at 161.29 50.8 0)
       (effects (font (size 1.27 1.27)) (justify left bottom) hide)
     )
@@
     (pin "1")
   )
-  (symbol (lib_name "1N5060GP_1") (lib_id "1N5060GP:1N5060GP") (at 180.34 36.83 90) (unit 1)
+  (symbol (lib_name "1N5060GP_1") (lib_id "spectrum analyzer:1N5060GP") (at 180.34 36.83 90) (unit 1)
     (in_bom yes) (on_board yes) (fields_autoplaced)
     (property "Reference" "D1101" (id 0) (at 184.15 35.5599 90)
@@
       (effects (font (size 1.27 1.27)) (justify right))
     )
-    (property "Footprint" "Diode_THT:D_DO-41_SOD81_P7.62mm_Horizontal" (id 2) (at 180.34 36.83 0)
+    (property "Footprint" "DO15-12" (id 2) (at 182.88 44.45 0)
       (effects (font (size 1.27 1.27)) (justify left bottom) hide)
     )
@@
     (pin "1")
   )
-  (symbol (lib_name "1N5060GP_2") (lib_id "1N5060GP:1N5060GP") (at 217.17 36.83 90) (unit 1)
+  (symbol (lib_name "1N5060GP_2") (lib_id "spectrum analyzer:1N5060GP") (at 217.17 36.83 90) (unit 1)
     (in_bom yes) (on_board yes) (fields_autoplaced)
     (property "Reference" "D1103" (id 0) (at 220.98 35.5599 90)
@@
       (effects (font (size 1.27 1.27)) (justify right))
     )
-    (property "Footprint" "Diode_THT:D_DO-41_SOD81_P7.62mm_Horizontal" (id 2) (at 217.17 36.83 0)
+    (property "Footprint" "DO15-12" (id 2) (at 219.71 44.45 0)
       (effects (font (size 1.27 1.27)) (justify left bottom) hide)
     )
@@
     (pin "2")
   )
-  (symbol (lib_id "terminal-block:691103110003") (at 250.19 130.81 270) (unit 1)
+  (symbol (lib_id "spectrum analyzer:691103110003") (at 250.19 130.81 270) (unit 1)
     (in_bom yes) (on_board yes) (fields_autoplaced)
     (property "Reference" "J1102" (id 0) (at 251.46 129.5399 90)
@@
       (effects (font (size 1.27 1.27)) (justify left))
     )
-    (property "Footprint" "15v-supply:terminal-block-691103110003" (id 2) (at 250.19 130.81 0)
-      (effects (font (size 1.27 1.27)) (justify left bottom) hide)
-    )
+    (property "Footprint" "691103110003" (id 2) (at 250.19 130.81 0)
+      (effects (font (size 1.27 1.27)) (justify left bottom) hide)
+    )

Commit message: v7 conversion
Parts:
- D1101, D1102, D1103, D1104: Spice_Lib_File 15v-supply-spice/1n5060.lib -> (none); Spice_Model 1N5060 -> (none); Spice_Netlist_Enabled Y -> (none); Spice_Node_Sequence 2 1 -> (none); Spice_Primitive D -> (none)
- F1101: Spice_Model .1 -> (none); Spice_Netlist_Enabled Y -> (none); Spice_Primitive R -> (none)
- J1101, J1102: Spice_Model Terminal Block -> (none); Spice_Netlist_Enabled N -> (none); Spice_Primitive J -> (none)
- P1101: Spice_Model sin(0 120 60) -> (none); Spice_Netlist_Enabled Y -> (none); Spice_Primitive V -> (none)
- SW1101: value SW_SPST -> 0; Spice_Model dc 0 -> (none); Spice_Netlist_Enabled Y -> (none); Spice_Primitive V -> (none)
- T1101: Spice_Lib_File 15v-supply-spice/xformer.lib -> (none); Spice_Model XFORMER -> (none); Spice_Netlist_Enabled Y -> (none); Spice_Primitive X -> (none)
- U1101: Spice_Lib_File 15v-supply-spice/regulators.lib -> (none); Spice_Model LM7815 -> (none); Spice_Netlist_Enabled Y -> (none); Spice_Primitive X -> (none)
- U1102: Spice_Lib_File 15v-supply-spice/regulators.lib -> (none); Spice_Model LM7915 -> (none); Spice_Netlist_Enabled Y -> (none); Spice_Node_Sequence 2 1 3 -> (none); Spice_Primitive X -> (none)
