File: hierarchical-schematic/70mhz-lpfilter.kicad_sch (KiCad schematic)
At the start: 11 parts, among them J701 Coax Solder Point, J702 Coax Solder Point

Commit message: appearance improvements
Parts:
- J701: value Coax Solder Point -> In
- J702: value Coax Solder Point -> Out
Changed lines of the file:
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@@
   (junction (at 113.03 113.03) (diameter 0) (color 0 0 0 0)
   )
+  (junction (at 232.41 113.03) (diameter 0) (color 0 0 0 0)
+  )
   (junction (at 224.79 113.03) (diameter 0) (color 0 0 0 0)
   )
@@
     (stroke (width 0) (type default) (color 0 0 0 0))
   )
+  (wire (pts (xy 232.41 113.03) (xy 232.41 102.87))
+    (stroke (width 0) (type default) (color 0 0 0 0))
+  )
   (wire (pts (xy 199.39 118.11) (xy 199.39 113.03))
     (stroke (width 0) (type default) (color 0 0 0 0))
@@
     (stroke (width 0) (type default) (color 0 0 0 0))
   )
-  (wire (pts (xy 90.17 100.33) (xy 113.03 100.33))
+  (wire (pts (xy 107.95 100.33) (xy 113.03 100.33))
     (stroke (width 0) (type default) (color 0 0 0 0))
   )
@@
     (stroke (width 0) (type default) (color 0 0 0 0))
   )
+  (wire (pts (xy 232.41 102.87) (xy 236.22 102.87))
+    (stroke (width 0) (type default) (color 0 0 0 0))
+  )
   (wire (pts (xy 199.39 125.73) (xy 199.39 123.19))
     (stroke (width 0) (type default) (color 0 0 0 0))
@@
     (stroke (width 0) (type default) (color 0 0 0 0))
   )
-  (hierarchical_label "70Mhz LP Filter Signal" (shape input) (at 229.87 113.03 90)
+  (hierarchical_label "70Mhz LP Filter Signal" (shape input) (at 236.22 102.87 0)
     (effects (font (size 1.27 1.27)) (justify left))
   )
-  (hierarchical_label "Signal In" (shape input) (at 90.17 100.33 180)
+  (hierarchical_label "Signal In" (shape input) (at 107.95 100.33 180)
     (effects (font (size 1.27 1.27)) (justify right))
   )
@@
     (in_bom yes) (on_board yes) (fields_autoplaced)
     (property "Reference" "J701" (id 0) (at 108.2674 105.41 0))
-    (property "Value" "Coax Solder Point" (id 1) (at 108.2674 107.95 0))
+    (property "Value" "In" (id 1) (at 108.2674 107.95 0))
     (property "Footprint" "Connector_Wire:SolderWire-0.5sqmm_1x02_P4.6mm_D0.9mm_OD2.1mm" (id 2) (at 107.95 113.03 0)
       (effects (font (size 1.27 1.27)) hide)
@@
       (effects (font (size 1.27 1.27)) (justify left))
     )
-    (property "Value" "Coax Solder Point" (id 1) (at 240.03 114.5931 0)
-      (effects (font (size 1.27 1.27)) (justify left))
-    )
+    (property "Value" "Out" (id 1) (at 240.03 114.5931 0)
+      (effects (font (size 1.27 1.27)) (justify left))
+    )

Commit message: v7 conversion
Parts:
- J701, J702: Spice_Model Conn_Coaxial -> (none); Spice_Netlist_Enabled N -> (none); Spice_Primitive J -> (none)
