File: hierarchical-schematic/110_7mhz-filter.kicad_sch (KiCad schematic)
At the start: 12 parts, among them J601 In, J602 Out

Commit message: appearance improvements
Other:
- moved on the sheet: C603, C605
Changed lines of the file:
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@@
   (junction (at 127 113.03) (diameter 0) (color 0 0 0 0)
+  )
+  (junction (at 236.22 113.03) (diameter 0) (color 0 0 0 0)
   )
   (junction (at 228.6 113.03) (diameter 0) (color 0 0 0 0)
@@
   )
   (junction (at 182.88 113.03) (diameter 0) (color 0 0 0 0)
+  )
+  (junction (at 119.38 113.03) (diameter 0) (color 0 0 0 0)
   )
   (junction (at 152.4 113.03) (diameter 0) (color 0 0 0 0)
@@
     (stroke (width 0) (type default) (color 0 0 0 0))
   )
+  (wire (pts (xy 241.3 101.6) (xy 236.22 101.6))
+    (stroke (width 0) (type default) (color 0 0 0 0))
+  )
   (wire (pts (xy 218.44 113.03) (xy 228.6 113.03))
     (stroke (width 0) (type default) (color 0 0 0 0))
@@
     (stroke (width 0) (type default) (color 0 0 0 0))
   )
-  (wire (pts (xy 167.64 113.03) (xy 171.45 113.03))
+  (wire (pts (xy 165.1 113.03) (xy 171.45 113.03))
     (stroke (width 0) (type default) (color 0 0 0 0))
   )
@@
     (stroke (width 0) (type default) (color 0 0 0 0))
   )
-  (wire (pts (xy 193.04 113.03) (xy 203.2 113.03))
+  (wire (pts (xy 195.58 113.03) (xy 203.2 113.03))
+    (stroke (width 0) (type default) (color 0 0 0 0))
+  )
+  (wire (pts (xy 114.3 101.6) (xy 119.38 101.6))
     (stroke (width 0) (type default) (color 0 0 0 0))
   )
@@
     (stroke (width 0) (type default) (color 0 0 0 0))
   )
+  (wire (pts (xy 236.22 101.6) (xy 236.22 113.03))
+    (stroke (width 0) (type default) (color 0 0 0 0))
+  )
   (wire (pts (xy 114.3 128.27) (xy 114.3 118.11))
+    (stroke (width 0) (type default) (color 0 0 0 0))
+  )
+  (wire (pts (xy 119.38 101.6) (xy 119.38 113.03))
     (stroke (width 0) (type default) (color 0 0 0 0))
   )
@@
     (stroke (width 0) (type default) (color 0 0 0 0))
   )
-  (wire (pts (xy 182.88 113.03) (xy 187.96 113.03))
+  (wire (pts (xy 182.88 113.03) (xy 190.5 113.03))
     (stroke (width 0) (type default) (color 0 0 0 0))
   )
@@
     (stroke (width 0) (type default) (color 0 0 0 0))
   )
-  (wire (pts (xy 152.4 113.03) (xy 162.56 113.03))
+  (wire (pts (xy 152.4 113.03) (xy 160.02 113.03))
     (stroke (width 0) (type default) (color 0 0 0 0))
   )
-  (hierarchical_label "1st IF" (shape input) (at 121.92 113.03 90)
-    (effects (font (size 1.27 1.27)) (justify left))
+  (hierarchical_label "1st IF" (shape input) (at 114.3 101.6 180)
+    (effects (font (size 1.27 1.27)) (justify right))
   )
-  (hierarchical_label "110MHz Filter" (shape output) (at 233.68 113.03 90)
+  (hierarchical_label "110MHz Filter" (shape output) (at 241.3 101.6 0)
     (effects (font (size 1.27 1.27)) (justify left))
   )
@@
     (pin "1")
   )
-  (symbol (lib_id "Device:C_Small") (at 165.1 113.03 90) (unit 1)
+  (symbol (lib_id "Device:C_Small") (at 162.56 113.03 90) (unit 1)
     (in_bom yes) (on_board yes) (fields_autoplaced)
-    (property "Reference" "C603" (id 0) (at 165.1063 106.68 90))
-    (property "Value" ".092p" (id 1) (at 165.1063 109.22 90))
-    (property "Footprint" "" (id 2) (at 165.1 113.03 0)
+    (property "Reference" "C603" (id 0) (at 162.5663 106.68 90))
+    (property "Value" ".092p" (id 1) (at 162.5663 109.22 90))
+    (property "Footprint" "" (id 2) (at 162.56 113.03 0)
       (effects (font (size 1.27 1.27)) hide)
     )
-    (property "Datasheet" "~" (id 3) (at 165.1 113.03 0)
+    (property "Datasheet" "~" (id 3) (at 162.56 113.03 0)
       (effects (font (size 1.27 1.27)) hide)
     )
@@
     (pin "1")
   )
-  (symbol (lib_id "Device:C_Small") (at 190.5 113.03 90) (unit 1)
+  (symbol (lib_id "Device:C_Small") (at 193.04 113.03 90) (unit 1)
     (in_bom yes) (on_board yes) (fields_autoplaced)
-    (property "Reference" "C605" (id 0) (at 190.5063 106.68 90))
-    (property "Value" ".092p" (id 1) (at 190.5063 109.22 90))
-    (property "Footprint" "" (id 2) (at 190.5 113.03 0)
+    (property "Reference" "C605" (id 0) (at 193.0463 106.68 90))
+    (property "Value" ".092p" (id 1) (at 193.0463 109.22 90))
+    (property "Footprint" "" (id 2) (at 193.04 113.03 0)
       (effects (font (size 1.27 1.27)) hide)
     )
-    (property "Datasheet" "~" (id 3) (at 190.5 113.03 0)
+    (property "Datasheet" "~" (id 3) (at 193.04 113.03 0)
       (effects (font (size 1.27 1.27)) hide)
     )
